File: Parts.kicad_sch (KiCad schematic)
At the start: 18 parts, among them J2 AudioJack3, J3 Conn_01x05, Q1 AO3400A, Q101 SI2302, U1 ESP32-DEVKITC-32D, U103 LMV358AIDR

Commit message: update some
Parts:
- added C5: 10u, Capacitor_SMD:C_1206_3216Metric_Pad1.33x1.80mm_HandSolder, symbol Device:C
- added D1: RED, symbol Device:LED
- added LED3: 19-217/GHC-YR1S2/3T, LED_SMD:LED_0603_1608Metric_Pad1.05x0.95mm_HandSolder, symbol Device:LED
- added P1: TLP291(GB-TP,SE, mylib:TLP291, symbol Isolator:SFH617A-1
- added R111: 10k, Resistor_SMD:R_0402_1005Metric, symbol Device:R
- added R2, R3: 220 0.25W, Resistor_SMD:R_1206_3216Metric_Pad1.30x1.75mm_HandSolder, symbol Device:R
- added R4: 1k, Resistor_SMD:R_0402_1005Metric, symbol Device:R
- added R8: 5.1k, Resistor_SMD:R_0402_1005Metric, symbol Device:R
- added U2: 74HC14, Package_SO:TSSOP-14_4.4x5mm_P0.65mm, symbol 74xx:74HC14
- added U7: TLP2361_TPL_E, Package_SO:SO-5_4.4x3.6mm_P1.27mm, symbol MIDI-Interface-san-rescue:TLP2361_TPL_E-dk_Optoisolators-Logic-Output
- added USB1: USB_C_Receptacle, Connector_USB:USB_C_Receptacle_HCTL_HC-TYPE-C-16P-01A, symbol Connector:USB_C_Receptacle
Connections:
- new net: USB1.A4 (VBUS), USB1.A9 (VBUS), USB1.B4 (VBUS), USB1.B9 (VBUS)
- new net GND: USB1.A1 (GND), USB1.A12 (GND), USB1.B1 (GND), USB1.B12 (GND)
- no-connect marks 1 -> 2
Other:
- note added: "0402 (Basic)"
- note added: "1206 extended For MIDI"
- note added: "50V X5R 1206 Basic"
- note added: "Robust"
- note added: "green"
- note added: "standard"
- moved on the sheet: R110
